Commit message: Integrated robot into Gazebo, no controls available

File: rs_description/urdf/basic/basic-rs.urdf (robot description, URDF)
Before this commit: robot basic-rocke, 1 links, 0 joints
Links:
- added link dummy
- link base_link: mass None -> ${chasis_mass}; geometry collision box size=${chasis_width} ${chasis_length} ${chasis_height}; visual box size=${chasis_width} ${chasis_length} ${chasis_height}
Joints:
- added joint dummy_joint: type fixed, parent dummy, child base_link
