Commit message: Rover mounted with sensors

File: rs_description/urdf_v2/rover/rover.xacro (robot description, xacro)
@@ -1,18 +1,17 @@
 <robot xmlns:xacro="http://www.ros.org/wiki/xacro" name="robot_name">
-    <link name="base_link_rover" />
+    <link name="base_link" />
     <xacro:include filename="$(find rs_description)/urdf_v2/rover_movement/rover_movement.xacro"/>
     <!-- <xacro:include filename="$(find rover_description)/urdf/rover_manipulator/rover_manipulator.xacro"/> -->
-    <!-- <xacro:include filename="$(find realsense2_description)/urdf/test_d435_camera.urdf.xacro"/> -->
+    <xacro:include filename="$(find rs_description)/urdf_v2/sensors/sensors.macro.xacro"/>
+    <xacro:include filename="$(find realsense2_description)/urdf/_d435.urdf.xacro" />
     <joint name="base_link_to_chassis" type="fixed">
-        <parent link="base_link_rover"/>
+        <parent link="base_link"/>
         <child link="chassis_link"/>
         <origin xyz="0 0 ${-chassis_height/2}" rpy="0 0 0"/>
     </joint>
-    <!-- <xacro:sensor_d435 name="sensor_d435"/>
-    <joint name="camera_to_chassis" type="fixed">
-        <parent link="base_link"/>
-        <child link="sensor_d435"/>
-        <origin xyz="0 0 ${-chassis_height/2}" rpy="0 0 0"/>
-    </joint> -->
+    <xacro:sensor_d435 name="camera" topics_ns="camera" parent="base_link" publish_pointcloud="true">
+        <origin xyz="0 0 0" rpy="0 0 -1.5708" />
+    </xacro:sensor_d435>
+    <xacro:imu parent="base_link"/>
     <!-- <joint name="base_link_to_manipulator_link_joint" type="fixed">
         <origin xyz="0 0.23 0" rpy="0 0 ${PI}"/>
@@ -20,8 +19,3 @@
         <child link="manipulator_link"/>
     </joint> -->
-    <!-- <gazebo>
-        <plugin name="gazebo_ros_control" filename="libgazebo_ros_control.so">
-            <robotNamespace>/</robotNamespace>
-        </plugin>
-    </gazebo> -->
 </robot>

File: rs_description/urdf_v2/rover_manipulator/rover_manipulator.xacro (robot description, xacro)
@@ -12,5 +12,5 @@
       <origin xyz="0 0 0" rpy="0 0 0"/>
       <geometry>
-        <mesh filename="package://rover_description/urdf/rover_manipulator/meshes/visual/manipulator_link.stl"/>
+        <mesh filename="package://rs_description/urdf_v2/rover_manipulator/meshes/visual/manipulator_link.stl"/>
       </geometry>
       <material name="white"/>
@@ -26,5 +26,5 @@
       <origin xyz="0 0 0" rpy="0 0 0"/>
       <geometry>
-        <mesh filename="package://rover_description/urdf/rover_manipulator/meshes/visual/shoulder_pan_link.stl"/>
+        <mesh filename="package://rs_description/urdf_v2/rover_manipulator/meshes/visual/shoulder_pan_link.stl"/>
       </geometry>
       <material name="black"/>
@@ -40,5 +40,5 @@
       <origin xyz="0 0 0" rpy="0 0 0"/>
       <geometry>
-        <mesh filename="package://rover_description/urdf/rover_manipulator/meshes/visual/shoulder_tilt_link.stl"/>
+        <mesh filename="package://rs_description/urdf_v2/rover_manipulator/meshes/visual/shoulder_tilt_link.stl"/>
       </geometry>
       <material name="grey"/>
@@ -54,5 +54,5 @@
       <origin xyz="0 0 0" rpy="0 0 0"/>
       <geometry>
-        <mesh filename="package://rover_description/urdf/rover_manipulator/meshes/visual/elbow_tilt_link.stl"/>
+        <mesh filename="package://rs_description/urdf_v2/rover_manipulator/meshes/visual/elbow_tilt_link.stl"/>
       </geometry>
       <material name="grey"/>
@@ -68,5 +68,5 @@
       <origin xyz="0 0 0" rpy="0 0 0"/>
       <geometry>
-        <mesh filename="package://rover_description/urdf/rover_manipulator/meshes/visual/wrist_tilt_link.stl"/>
+        <mesh filename="package://rs_description/urdf_v2/rover_manipulator/meshes/visual/wrist_tilt_link.stl"/>
       </geometry>
       <material name="black"/>
@@ -82,5 +82,5 @@
       <origin xyz="0 0 0" rpy="0 0 0"/>
       <geometry>
-        <mesh filename="package://rover_description/urdf/rover_manipulator/meshes/visual/wrist_yaw_link.stl"/>
+        <mesh filename="package://rs_description/urdf_v2/rover_manipulator/meshes/visual/wrist_yaw_link.stl"/>
       </geometry>
       <material name="grey"/>
@@ -96,5 +96,5 @@
       <origin xyz="0 0 0" rpy="0 0 0"/>
       <geometry>
-        <mesh filename="package://rover_description/urdf/rover_manipulator/meshes/visual/l_gripper_inner_link.stl"/>
+        <mesh filename="package://rs_description/urdf_v2/rover_manipulator/meshes/visual/l_gripper_inner_link.stl"/>
       </geometry>
       <material name="black"/>
@@ -110,5 +110,5 @@
       <origin xyz="0 0 0" rpy="0 0 0"/>
       <geometry>
-        <mesh filename="package://rover_description/urdf/rover_manipulator/meshes/visual/l_gripper_outer_link.stl"/>
+        <mesh filename="package://rs_description/urdf_v2/rover_manipulator/meshes/visual/l_gripper_outer_link.stl"/>
       </geometry>
       <material name="black"/>
@@ -124,5 +124,5 @@
       <origin xyz="0 0 0" rpy="0 0 0"/>
       <geometry>
-        <mesh filename="package://rover_description/urdf/rover_manipulator/meshes/visual/l_finger_link.stl"/>
+        <mesh filename="package://rs_description/urdf_v2/rover_manipulator/meshes/visual/l_finger_link.stl"/>
       </geometry>
       <material name="grey"/>
@@ -138,5 +138,5 @@
       <origin xyz="0 0 0" rpy="0 ${PI} 0"/>
       <geometry>
-        <mesh filename="package://rover_description/urdf/rover_manipulator/meshes/visual/r_gripper_inner_link.stl"/>
+        <mesh filename="package://rs_description/urdf_v2/rover_manipulator/meshes/visual/r_gripper_inner_link.stl"/>
       </geometry>
       <material name="black"/>
@@ -152,5 +152,5 @@
       <origin xyz="0 0 0" rpy="0 0 0"/>
       <geometry>
-        <mesh filename="package://rover_description/urdf/rover_manipulator/meshes/visual/r_gripper_outer_link.stl"/>
+        <mesh filename="package://rs_description/urdf_v2/rover_manipulator/meshes/visual/r_gripper_outer_link.stl"/>
       </geometry>
       <material name="black"/>
@@ -166,5 +166,5 @@
       <origin xyz="0 0 0" rpy="0 0 0"/>
       <geometry>
-        <mesh filename="package://rover_description/urdf/rover_manipulator/meshes/visual/r_finger_link.stl"/>
+        <mesh filename="package://rs_description/urdf_v2/rover_manipulator/meshes/visual/r_finger_link.stl"/>
       </geometry>
       <material name="grey"/>

File: rs_description/urdf_v2/rover_movement/rover_movement.xacro (robot description, xacro)
@@ -9,10 +9,10 @@
             <origin rpy="0 0 0" xyz="0 0 0"/>
             <geometry>
-                <mesh filename="package://rover_description/urdf/rover_movement/meshes/chassis.dae"/>
+                <mesh filename="package://rs_description/urdf_v2/rover_movement/meshes/chassis.dae"/>
             </geometry>
         </visual>
         <collision>
                 <geometry>
-                    <!-- <mesh filename="package://rover_description/urdf/rover_movement/meshes/sway_pivot.dae"/> -->
+                    <!-- <mesh filename="package://rs_description/urdf_v2/rover_movement/meshes/sway_pivot.dae"/> -->
                     <box size="${chassis_width} ${chassis_length} ${chassis_height}"/>
                 </geometry>
@@ -27,17 +27,17 @@
     <xacro:swaypivot name="l" lr="${left}" />
     <xacro:swaypivot name="r" lr="${right}" />
-    <joint name="l_swaypivot_joint" type="revolute">
+    <joint name="l_swaypivot_joint" type="fixed">
         <parent link="chassis_link"/>
         <child link="l_swaypivot_link"/>
         <origin xyz="${1*(chassis_width/2 + sway_pivot_depth/2 + sway_pivot_gap)} 0.0 0.0" rpy="0 0 0"/>
         <axis xyz="1.0 0.0 0.0"/>
-        <limit effort="1000" velocity="1000" lower="${-pi * 0.25}" upper="${pi * 0.25}"/>
+        <!-- <limit effort="1000" velocity="1000" lower="${-pi * 0.25}" upper="${pi * 0.25}"/> -->
     </joint>
-    <joint name="r_swaypivot_joint" type="revolute">
+    <joint name="r_swaypivot_joint" type="fixed">
         <parent link="chassis_link"/>
         <child link="r_swaypivot_link"/>
         <origin xyz="${-1*(chassis_width/2 + sway_pivot_depth/2 + sway_pivot_gap)} 0.0 0.0" rpy="0 0 0"/>
         <axis xyz="1.0 0.0 0.0"/>
-        <limit effort="1000" velocity="1000" lower="${-pi * 0.25}" upper="${pi * 0.25}"/>
+        <!-- <limit effort="1000" velocity="1000" lower="${-pi * 0.25}" upper="${pi * 0.25}"/> -->
         <mimic joint="l_swaypivot_joint" multiplier="-1" offset="0"/>
     </joint>

File: rs_description/urdf_v2/rover_movement/utils/macros.xacro (robot description, xacro)
@@ -5,5 +5,5 @@
             <visual>
                 <geometry>
-                    <mesh filename="package://rover_description/urdf/rover_movement/meshes/sway_pivot.dae"/>
+                    <mesh filename="package://rs_description/urdf_v2/rover_movement/meshes/sway_pivot.dae"/>
                 </geometry>
                 <origin xyz="0 0 0" rpy="0 0 ${lr*pi/2}"/>
@@ -33,5 +33,5 @@
             <visual>
                 <geometry>
-                    <mesh filename="package://rover_description/urdf/rover_movement/meshes/bottom_link.dae"/>
+                    <mesh filename="package://rs_description/urdf_v2/rover_movement/meshes/bottom_link.dae"/>
                 </geometry>
                 <origin xyz="0 0 0" rpy="0 0 ${fb*pi/2}"/>
@@ -49,5 +49,5 @@
             </inertial>
         </link>
-        <joint name="${sway}_swaypivot_${name}_upper_leg_joint" type="revolute">
+        <joint name="${sway}_swaypivot_${name}_upper_leg_joint" type="fixed">
             <parent link="${sway}_swaypivot_link"/>
             <child link="${name}_leg_link"/>
@@ -55,11 +55,11 @@
             <axis xyz="${-fb*1.0} 0 0"/>
             <!-- TODO: set variables to these limits -->
-            <limit effort="1000" velocity="1000" lower="-0.2" upper="0.65"/>
-            <dynamics damping="50" friction="1"/>
+            <!-- <limit effort="1000" velocity="1000" lower="-0.2" upper="0.65"/> -->
+            <!-- <dynamics damping="50" friction="1"/> -->
         </joint>
         <link name="${name}_upper_leg_mimic_link">
             <visual>
                 <geometry>
-                    <mesh filename="package://rover_description/urdf/rover_movement/meshes/top_link.dae"/>
+                    <mesh filename="package://rs_description/urdf_v2/rover_movement/meshes/top_link.dae"/>
                 </geometry>
                 <origin xyz="0 0 0" rpy="0 0 ${fb*pi/2}"/>
@@ -77,5 +77,5 @@
             </inertial>
         </link>
-        <joint name="${sway}_swaypivot_${name}_upper_leg_mimic_joint" type="revolute">
+        <joint name="${sway}_swaypivot_${name}_upper_leg_mimic_joint" type="fixed">
             <parent link="${sway}_swaypivot_link"/>
             <child link="${name}_upper_leg_mimic_link"/>
@@ -83,5 +83,5 @@
             <axis xyz="${-fb*1.0} 0 0"/>
             <!-- dont change these limits -->
-            <limit effort="1000" velocity="1000" lower="-10" upper="10"/>
+            <!-- <limit effort="1000" velocity="1000" lower="-10" upper="10"/> -->
             <mimic joint="${sway}_swaypivot_${name}_upper_leg_joint" multiplier="1" offset="0"/>
         </joint>
@@ -89,5 +89,5 @@
             <visual>
                 <geometry>
-                    <mesh filename="package://rover_description/urdf/rover_movement/meshes/parallel_link.dae"/>
+                    <mesh filename="package://rs_description/urdf_v2/rover_movement/meshes/parallel_link.dae"/>
                 </geometry>
                 <origin xyz="0 0 0" rpy="0 0 ${fb*pi/2}"/>
@@ -106,5 +106,5 @@
             </inertial>
         </link>
-        <joint name="${name}_leg_to_${name}_steer_hub_joint" type="revolute">
+        <joint name="${name}_leg_to_${name}_steer_hub_joint" type="fixed">
             <parent link="${name}_leg_link"/>
             <child link="${name}_steer_hub_link"/>
@@ -112,12 +112,12 @@
             <axis xyz="${-fb*1.0} 0 0"/>
             <!-- dont change these limits -->
-            <limit effort="1000" velocity="1000" lower="-10" upper="10"/>
-            <mimic joint="${sway}_swaypivot_${name}_upper_leg_joint" multiplier="-1" offset="0"/>
-            <dynamics damping="50" friction="1"/>
+            <!-- <limit effort="1000" velocity="1000" lower="-10" upper="10"/> -->
+            <!-- <mimic joint="${sway}_swaypivot_${name}_upper_leg_joint" multiplier="-1" offset="0"/> -->
+            <!-- <dynamics damping="50" friction="1"/> -->
         </joint>
         <link name="${name}_steer_link">
             <visual>
                 <geometry>
-                    <mesh filename="package://rover_description/urdf/rover_movement/meshes/steer_hub.dae"/>
+                    <mesh filename="package://rs_description/urdf_v2/rover_movement/meshes/steer_hub.dae"/>
                 </geometry>
                 <origin xyz="0 0 0" rpy="0 ${pi} ${wheel_config*lr*pi/2}"/>
@@ -137,5 +137,5 @@
             </inertial>
         </link>
-        <joint name="${name}_leg_to_${name}_steer_joint" type="revolute">
+        <joint name="${name}_leg_to_${name}_steer_joint" type="fixed">
             <parent link="${name}_steer_hub_link"/>
             <child link="${name}_steer_link"/>
@@ -143,11 +143,11 @@
             <axis xyz="0 0 ${fb*lr*1.0}"/>
             <!-- dont change these limits -->
-            <limit effort="1000" velocity="1000" lower="${-2*pi}" upper="${2*pi}"/>
-            <dynamics damping="50" friction="1"/>
+            <!-- <limit effort="1000" velocity="1000" lower="${-2*pi}" upper="${2*pi}"/> -->
+            <!-- <dynamics damping="50" friction="1"/> -->
         </joint>
         <link name="${name}_wheel_link">
             <visual>
                 <geometry>
-                    <mesh filename="package://rover_description/urdf/rover_movement/meshes/wheel.dae"/>
+                    <mesh filename="package://rs_description/urdf_v2/rover_movement/meshes/wheel.dae"/>
                 </geometry>
                 <origin xyz="0 0 0" rpy="0 0 ${wheel_config*lr*pi/2}"/>
@@ -168,5 +168,5 @@
             <parent link="${name}_steer_link"/>
             <child link="${name}_wheel_link"/>
-            <dynamics damping="50" friction="1"/>
+            <!-- <dynamics damping="50" friction="1"/> -->
         </joint>
         <transmission name="${name}_wheel_trans" type="SimpleTransmission">
@@ -179,5 +179,5 @@
             </joint>
         </transmission>
-        <transmission name="${name}_steering_trans" type="SimpleTransmission">
+        <!-- <transmission name="${name}_steering_trans" type="SimpleTransmission">
             <type>transmission_interface/SimpleTransmission</type>
             <actuator name="${name}_steering_motor">
@@ -188,5 +188,5 @@
                 <hardwareInterface>PositionJointInterface</hardwareInterface>
             </joint>
-        </transmission>
+        </transmission> -->
     </xacro:macro>
 </robot>
